File: Hardware/schematic/VC5_schematic/LEDs.kicad_sch (KiCad schematic)
At the start: 13 parts, among them Q1 BC337

Commit message: minor updates to the schematic
Parts:
- removed C1, C2, C3, C4, C5: 1u, symbol Device:C
- added C1, C2, C3, C4, C5: 1u, symbol Device:C_Polarized
Connections:
- net +5V: now also C1.1, C2.1, C3.1, C4.1, C5.1
- net GND: now also C1.2, C2.2, C3.2, C4.2, C5.2
Other:
- note added: "07.10.2024"
- note added: "1.0"
- note added: "Designed by Jan Eberhardt"
- note added: "Projekt "VC 5""

Commit message: added missing footprints, changed schematic symbols for the rotaries
Parts:
- C1, C2, C3, C4, C5: footprint (none) -> Capacitor_THT:CP_Radial_D4.0mm_P1.50mm
- R1, R2: footprint (none) -> Resistor_THT:R_Axial_DIN0207_L6.3mm_D2.5mm_P2.54mm_Vertical
Changed lines of the file:
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@@
 			)
 		)
-		(property "Footprint" ""
+		(property "Footprint" "Capacitor_THT:CP_Radial_D4.0mm_P1.50mm"
 			(at 133.35 73.3552 0)
 			(effects
@@
 			)
 		)
-		(property "Footprint" ""
+		(property "Footprint" "Capacitor_THT:CP_Radial_D4.0mm_P1.50mm"
 			(at 232.41 73.3552 0)
 			(effects
@@
 			)
 		)
-		(property "Footprint" ""
+		(property "Footprint" "Capacitor_THT:CP_Radial_D4.0mm_P1.50mm"
 			(at 100.33 73.3552 0)
 			(effects
@@
 			)
 		)
-		(property "Footprint" ""
+		(property "Footprint" "Capacitor_THT:CP_Radial_D4.0mm_P1.50mm"
 			(at 199.39 73.3552 0)
 			(effects
@@
 			)
 		)
-		(property "Footprint" ""
+		(property "Footprint" "Resistor_THT:R_Axial_DIN0207_L6.3mm_D2.5mm_P2.54mm_Vertical"
 			(at 88.392 76.2 90)
 			(effects
@@
 			)
 		)
-		(property "Footprint" ""
+		(property "Footprint" "Capacitor_THT:CP_Radial_D4.0mm_P1.50mm"
 			(at 166.37 73.3552 0)
 			(effects
@@
 			)
 		)
-		(property "Footprint" ""
+		(property "Footprint" "Resistor_THT:R_Axial_DIN0207_L6.3mm_D2.5mm_P2.54mm_Vertical"
 			(at 62.992 68.58 90)
 			(effects

Commit message: first layout
Parts:
- D1, D2, D3, D4, D5: footprint LED_THT:LED_D5.0mm-4_RGB -> WS2812_LED_THT:LED_D5.0mm-4_RGB
- Q1: footprint Package_TO_SOT_THT:TO-92_Inline -> Package_TO_SOT_THT:TO-92_Inline_Wide
- R1, R2: footprint Resistor_THT:R_Axial_DIN0207_L6.3mm_D2.5mm_P2.54mm_Vertical -> Resistor_THT:R_Axial_DIN0207_L6.3mm_D2.5mm_P10.16mm_Horizontal
Changed lines of the file:
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@@
 			)
 		)
-		(property "Footprint" "LED_THT:LED_D5.0mm-4_RGB"
+		(property "Footprint" "WS2812_LED_THT:LED_D5.0mm-4_RGB"
 			(at 177.8 95.25 0)
 			(effects
@@
 			)
 		)
-		(property "Footprint" "Package_TO_SOT_THT:TO-92_Inline"
+		(property "Footprint" "Package_TO_SOT_THT:TO-92_Inline_Wide"
 			(at 62.865 87.63 0)
 			(effects
@@
 			)
 		)
-		(property "Footprint" "LED_THT:LED_D5.0mm-4_RGB"
+		(property "Footprint" "WS2812_LED_THT:LED_D5.0mm-4_RGB"
 			(at 144.78 95.25 0)
 			(effects
@@
 			)
 		)
-		(property "Footprint" "LED_THT:LED_D5.0mm-4_RGB"
+		(property "Footprint" "WS2812_LED_THT:LED_D5.0mm-4_RGB"
 			(at 210.82 95.25 0)
 			(effects
@@
 			)
 		)
-		(property "Footprint" "LED_THT:LED_D5.0mm-4_RGB"
+		(property "Footprint" "WS2812_LED_THT:LED_D5.0mm-4_RGB"
 			(at 111.76 95.25 0)
 			(effects
@@
 			)
 		)
-		(property "Footprint" "LED_THT:LED_D5.0mm-4_RGB"
+		(property "Footprint" "WS2812_LED_THT:LED_D5.0mm-4_RGB"
 			(at 243.84 95.25 0)
 			(effects
@@
 			)
 		)
-		(property "Footprint" "Resistor_THT:R_Axial_DIN0207_L6.3mm_D2.5mm_P2.54mm_Vertical"
+		(property "Footprint" "Resistor_THT:R_Axial_DIN0207_L6.3mm_D2.5mm_P10.16mm_Horizontal"
 			(at 88.392 76.2 90)
 			(effects
@@
 			)
 		)
-		(property "Footprint" "Resistor_THT:R_Axial_DIN0207_L6.3mm_D2.5mm_P2.54mm_Vertical"
+		(property "Footprint" "Resistor_THT:R_Axial_DIN0207_L6.3mm_D2.5mm_P10.16mm_Horizontal"
 			(at 62.992 68.58 90)
 			(effects

Commit message: reworked the PCB layout
Connections:
- net at D3.1 (DO): now also D2.4 (DI); no longer D4.4 (DI)
- net at D2.1 (DO): now also D1.4 (DI); no longer D3.4 (DI)
- net at Q1.1 (C), R2.2: now also D5.4 (DI); no longer D1.4 (DI)
- net at D1.1 (DO): no longer D2.4 (DI)
- net at D4.1 (DO): now also D3.4 (DI); no longer D5.4 (DI)
- net at D5.1 (DO): now also D4.4 (DI)
