File: Hardware/schematic/VC5_schematic/displays.kicad_sch (KiCad schematic)
At the start: 5 parts

Commit message: updated display values
Parts:
- U2, U3, U4, U5, U6: value ~ -> 1.3in SH1106 OLED
Changed lines of the file:
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@@
 		(on_board yes)
 		(dnp no)
-		(fields_autoplaced yes)
 		(property "Reference" "U5"
 			(at 196.85 59.0549 0)
@@
 			)
 		)
-		(property "Value" "~"
-			(at 196.85 60.96 0)
+		(property "Value" "1.3in SH1106 OLED"
+			(at 174.752 53.594 0)
 			(effects
 				(font
@@
 		(on_board yes)
 		(dnp no)
-		(fields_autoplaced yes)
 		(property "Reference" "U3"
 			(at 124.46 59.0549 0)
@@
 			)
 		)
-		(property "Value" "~"
-			(at 124.46 60.96 0)
+		(property "Value" "1.3in SH1106 OLED"
+			(at 101.854 53.34 0)
 			(effects
 				(font
@@
 		(on_board yes)
 		(dnp no)
-		(fields_autoplaced yes)
 		(property "Reference" "U4"
 			(at 160.02 59.0549 0)
@@
 			)
 		)
-		(property "Value" "~"
-			(at 160.02 60.96 0)
+		(property "Value" "1.3in SH1106 OLED"
+			(at 137.922 53.594 0)
 			(effects
 				(font
@@
 		(on_board yes)
 		(dnp no)
-		(fields_autoplaced yes)
 		(property "Reference" "U2"
 			(at 88.9 59.0549 0)
@@
 			)
 		)
-		(property "Value" "~"
-			(at 88.9 60.96 0)
+		(property "Value" "1.3in SH1106 OLED"
+			(at 66.548 53.086 0)
 			(effects
 				(font
@@
 		(on_board yes)
 		(dnp no)
-		(fields_autoplaced yes)
 		(property "Reference" "U6"
 			(at 233.68 59.0549 0)
@@
 			)
 		)
-		(property "Value" "~"
-			(at 233.68 60.96 0)
-			(effects
-				(font
+		(property "Value" "1.3in SH1106 OLED"
+			(at 211.328 53.594 0)
+			(effects
+				(font

Commit message: minor updates to the schematic
Connections:
- net reset_displays renamed DISP_RESET
Other:
- note added: "07.10.2024"
- note added: "1.0"
- note added: "Designed by Jan Eberhardt"
- note added: "Projekt "VC 5""
Changed lines of the file:
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@@
+		)
+	)
+	(text "Designed by Jan Eberhardt"
+		(exclude_from_sim no)
+		(at 193.802 168.402 0)
+		(effects
+			(font
+				(size 1.5 1.5)
+			)
+		)
+	)
+	(text "07.10.2024"
+		(exclude_from_sim no)
+		(at 213.614 193.294 0)
+		(effects
+			(font
+				(size 1.5 1.5)
+			)
+		)
+	)
+	(text "Projekt \"VC 5\""
+		(exclude_from_sim no)
+		(at 200.914 189.738 0)
+		(effects
+			(font
+				(size 2.5 2.5)
+			)
+		)
+	)
+	(text "1.0"
+		(exclude_from_sim no)
+		(at 270.764 193.294 0)
+		(effects
+			(font
+				(size 1.5 1.5)
+			)
 		)
 	)
@@
 		)
 	)
-	(label "reset_displays"
+	(label "DISP_RESET"
 		(at 66.04 105.41 270)
 		(fields_autoplaced yes)
@@
 		)
 	)
-	(global_label "reset_displays"
+	(global_label "DISP_RESET"
 		(shape input)
 		(at 66.04 127 270)
@@
 		)
 		(property "Intersheetrefs" "${INTERSHEET_REFS}"
-			(at 66.04 143.4108 90)
-			(effects
-				(font
+			(at 66.04 140.398 90)
+			(effects
+				(font

Commit message: added missing footprints, changed schematic symbols for the rotaries
Parts:
- U2, U3, U4, U5, U6: footprint (none) -> Waveshare_displays:WaveShare_1in3_OLED_SH1106
Changed lines of the file:
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@@
 			)
 		)
-		(property "Footprint" ""
+		(property "Footprint" "Waveshare_displays:WaveShare_1in3_OLED_SH1106"
 			(at 196.85 57.15 0)
 			(effects
@@
 			)
 		)
-		(property "Datasheet" ""
+		(property "Datasheet" "https://www.waveshare.com/wiki/1.3inch_OLED_(B)#Overview"
 			(at 196.85 57.15 0)
 			(effects
@@
 			)
 		)
-		(property "Footprint" ""
+		(property "Footprint" "Waveshare_displays:WaveShare_1in3_OLED_SH1106"
 			(at 124.46 57.15 0)
 			(effects
@@
 			)
 		)
-		(property "Datasheet" ""
+		(property "Datasheet" "https://www.waveshare.com/wiki/1.3inch_OLED_(B)#Overview"
 			(at 124.46 57.15 0)
 			(effects
@@
 			)
 		)
-		(property "Footprint" ""
+		(property "Footprint" "Waveshare_displays:WaveShare_1in3_OLED_SH1106"
 			(at 160.02 57.15 0)
 			(effects
@@
 			)
 		)
-		(property "Datasheet" ""
+		(property "Datasheet" "https://www.waveshare.com/wiki/1.3inch_OLED_(B)#Overview"
 			(at 160.02 57.15 0)
 			(effects
@@
 			)
 		)
-		(property "Footprint" ""
+		(property "Footprint" "Waveshare_displays:WaveShare_1in3_OLED_SH1106"
 			(at 88.9 57.15 0)
 			(effects
@@
 			)
 		)
-		(property "Datasheet" ""
+		(property "Datasheet" "https://www.waveshare.com/wiki/1.3inch_OLED_(B)#Overview"
 			(at 88.9 57.15 0)
 			(effects
@@
 			)
 		)
-		(property "Footprint" ""
+		(property "Footprint" "Waveshare_displays:WaveShare_1in3_OLED_SH1106"
 			(at 233.68 57.15 0)
 			(effects
@@
 			)
 		)
-		(property "Datasheet" ""
+		(property "Datasheet" "https://www.waveshare.com/wiki/1.3inch_OLED_(B)#Overview"
 			(at 233.68 57.15 0)
 			(effects
