File: Hardware/schematic/VC5_schematic/VC5_schematic.kicad_sch (KiCad schematic)
At the start: 4 parts, among them J1 Debug_output, J2 +5V, J3 GND, U1 Pico

Commit message: minor updates to the schematic
Parts:
- removed J1: Debug_output, symbol Connector:Conn_01x02_Pin
- removed J2: +5V, symbol Connector:Conn_01x01_Pin
- removed J3: GND, symbol Connector:Conn_01x01_Pin
- added J2: Debug_output, symbol Connector:Conn_01x02_Socket
Connections:
- net +5V: now also U1.40 (VBUS)
- net GND: now also J2.2 (Pin_2)
- net at U1.1 (GPIO0): now also J2.1 (Pin_1)
- net I²C-SCL renamed I2C_SCL
- net I²C-SDA renamed I2C_SDA
- net reset_MCP renamed MCP_RESET
- net reset_displays renamed DISP_RESET
- no-connect marks 20 -> 19
Other:
- note added: "07.10.2024"
- note added: "1.0"
- note added: "Designed by Jan Eberhardt"
- note added: "Projekt "VC 5""
Changed lines of the file:
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@@
 	(paper "A4")
-	(junction
-		(at 193.04 76.2)
-		(diameter 0)
-		(color 0 0 0 0)
-	)
 	(junction
 		(at 177.8 71.12)
@@
 	)
 	(no_connect
-		(at 173.99 71.12)
-	)
-	(no_connect
 		(at 138.43 86.36)
 	)
@@
 	(wire
 		(pts
-			(xy 193.04 71.12) (xy 193.04 76.2)
-		)
-		(stroke
-			(width 0)
-			(type default)
-		)
-	)
-	(wire
-		(pts
 			(xy 173.99 111.76) (xy 200.66 111.76)
 		)
@@
 	(wire
 		(pts
-			(xy 177.8 71.12) (xy 182.88 71.12)
-		)
-		(stroke
-			(width 0)
-			(type default)
-		)
-	)
-	(wire
-		(pts
 			(xy 193.04 77.47) (xy 193.04 76.2)
 		)
@@
 	(wire
 		(pts
+			(xy 173.99 71.12) (xy 177.8 71.12)
+		)
+		(stroke
+			(width 0)
+			(type default)
+		)
+	)
+	(wire
+		(pts
 			(xy 125.73 111.76) (xy 138.43 111.76)
 		)
@@
 		)
 	)
-	(label "reset_displays"
+	(text "Projekt \"VC 5\""
+		(exclude_from_sim no)
+		(at 200.66 189.738 0)
+		(effects
+			(font
+				(size 2.5 2.5)
+			)
+		)
+	)
+	(text "1.0"
+		(exclude_from_sim no)
+		(at 270.51 193.294 0)
+		(effects
+			(font
+				(size 1.5 1.5)
+			)
+		)
+	)
+	(text "Designed by Jan Eberhardt"
+		(exclude_from_sim no)
+		(at 193.548 168.402 0)
+		(effects
+			(font
+				(size 1.5 1.5)
+			)
+		)
+	)
+	(text "07.10.2024"
+		(exclude_from_sim no)
+		(at 213.36 193.294 0)
+		(effects
+			(font
+				(size 1.5 1.5)
+			)
+		)
+	)
+	(label "DISP_RESET"
 		(at 111.76 133.35 270)
 		(fields_autoplaced yes)
@@
 		)
 	)
-	(global_label "I²C-SCL"
+	(global_label "I2C_SCL"
 		(shape output)
 		(at 121.92 93.98 180)
@@
 		)
 		(property "Intersheetrefs" "${INTERSHEET_REFS}"
-			(at 111.0124 93.98 0)
-			(effects
-				(font
-					(size 1.27 1.27)
-				)
-				(justify right)
-				(hide yes)
-			)
-		)
-	)
-	(global_label "I²C-SDA"
+			(at 112.0295 93.98 0)
+			(effects
+				(font
+					(size 1.27 1.27)
+				)
+				(justify right)
+				(hide yes)
+			)
+		)
+	)
+	(global_label "I2C_SDA"
 		(shape output)
 		(at 121.92 91.44 180)
@@
 		)
 		(property "Intersheetrefs" "${INTERSHEET_REFS}"
-			(at 110.9519 91.44 0)
+			(at 111.969 91.44 0)
 			(effects
 				(font
@@
 		)
 	)
-	(global_label "reset_MCP"
+	(global_label "MCP_RESET"
 		(shape output)
 		(at 121.92 78.74 180)
@@
 		)
 		(property "Intersheetrefs" "${INTERSHEET_REFS}"
-			(at 109.2586 78.74 0)
+			(at 108.8849 78.74 0)
 			(effects
 				(font
@@
 		)
 	)
-	(global_label "reset_displays"
+	(global_label "DISP_RESET"
 		(shape output)
 		(at 111.76 148.59 270)
@@
 		)
 		(property "Intersheetrefs" "${INTERSHEET_REFS}"
-			(at 111.76 165.0008 90)
+			(at 111.76 161.988 90)
 			(effects
 				(font
@@
 				(justify right)
 				(hide yes)
-			)
-		)
-	)
-	(symbol
-		(lib_id "Connector:Conn_01x02_Pin")
-		(at 140.97 53.34 270)
-		(unit 1)
-		(exclude_from_sim no)
-		(in_bom yes)
-		(on_board yes)
-		(dnp no)
-		(fields_autoplaced yes)
-		(property "Reference" "J1"
-			(at 142.24 52.7049 90)
-			(effects
-				(font
-					(size 1.27 1.27)
-				)
-				(justify left)
-			)
-		)
-		(property "Value" "Debug_output"
-			(at 142.24 55.2449 90)
-			(effects
-				(font
-					(size 1.27 1.27)
-				)
-				(justify left)
-			)
-		)
-		(property "Footprint" ""
-			(at 140.97 53.34 0)
-			(effects
-				(font
-					(size 1.27 1.27)
-				)
-				(hide yes)
-			)
-		)
-		(property "Datasheet" "~"
-			(at 140.97 53.34 0)
-			(effects
-				(font
-					(size 1.27 1.27)
-				)
-				(hide yes)
-			)
-		)
-		(property "Description" "Generic connector, single row, 01x02, script generated"
-			(at 140.97 53.34 0)
-			(effects
-				(font
-					(size 1.27 1.27)
-				)
-				(hide yes)
-			)
-		)
-		(pin "2"
-		)
-		(pin "1"
-		)
-		(instances
-			(project "VC5_schematic"
-				(path "/236c86f4-0879-4356-88b2-65461f963bd6"
-					(reference "J1")
-					(unit 1)
-				)
 			)
 		)
@@
 	)
 	(symbol
+		(lib_id "Connector:Conn_01x02_Socket")
+		(at 138.43 53.34 90)
+		(unit 1)
+		(exclude_from_sim no)
+		(in_bom yes)
+		(on_board yes)
+		(dnp no)
+		(fields_autoplaced yes)
+		(property "Reference" "J2"
+			(at 142.24 52.7049 90)
+			(effects
+				(font
+					(size 1.27 1.27)
+				)
+				(justify right)
+			)
+		)
+		(property "Value" "Debug_output"
+			(at 142.24 55.2449 90)
+			(effects
+				(font
+					(size 1.27 1.27)
+				)
+				(justify right)
+			)
+		)
+		(property "Footprint" ""
+			(at 138.43 53.34 0)
+			(effects
+				(font
+					(size 1.27 1.27)
+				)
+				(hide yes)
+			)
+		)
+		(property "Datasheet" "~"
+			(at 138.43 53.34 0)
+			(effects
+				(font
+					(size 1.27 1.27)
+				)
+				(hide yes)
+			)
+		)
+		(property "Description" "Generic connector, single row, 01x02, script generated"
+			(at 138.43 53.34 0)
+			(effects
+				(font
+					(size 1.27 1.27)
+				)
+				(hide yes)
+			)
+		)
+		(pin "2"
+		)
+		(pin "1"
+		)
+		(instances
+			(project ""
+				(path "/236c86f4-0879-4356-88b2-65461f963bd6"
+					(reference "J2")
+					(unit 1)
+				)
+			)
+		)
+	)
+	(symbol
 		(lib_id "power:GND")
 		(at 138.43 114.3 270)
@@
 				(path "/236c86f4-0879-4356-88b2-65461f963bd6"
 					(reference "#PWR04")
-					(unit 1)
-				)
-			)
-		)
-	)
-	(symbol
-		(lib_id "Connector:Conn_01x01_Pin")
-		(at 182.88 66.04 270)
-		(unit 1)
-		(exclude_from_sim no)
-		(in_bom yes)
-		(on_board yes)
-		(dnp no)
-		(fields_autoplaced yes)
-		(property "Reference" "J2"
-			(at 184.15 65.4049 90)
-			(effects
-				(font
-					(size 1.27 1.27)
-				)
-				(justify left)
-			)
-		)
-		(property "Value" "+5V"
-			(at 184.15 67.9449 90)
-			(effects
-				(font
-					(size 1.27 1.27)
-				)
-				(justify left)
-			)
-		)
-		(property "Footprint" ""
-			(at 182.88 66.04 0)
-			(effects
-				(font
-					(size 1.27 1.27)
-				)
-				(hide yes)
-			)
-		)
-		(property "Datasheet" "~"
-			(at 182.88 66.04 0)
-			(effects
-				(font
-					(size 1.27 1.27)
-				)
-				(hide yes)
-			)
-		)
-		(property "Description" "Generic connector, single row, 01x01, script generated"
-			(at 182.88 66.04 0)
-			(effects
-				(font
-					(size 1.27 1.27)
-				)
-				(hide yes)
-			)
-		)
-		(pin "1"
-		)
-		(instances
-			(project "VC5_schematic"
-				(path "/236c86f4-0879-4356-88b2-65461f963bd6"
-					(reference "J2")
 					(unit 1)
 				)
@@
 					(unit 1)
 				)
-			)
-		)
-	)
-	(symbol
-		(lib_id "Connector:Conn_01x01_Pin")
-		(at 193.04 66.04 270)
-		(unit 1)
-		(exclude_from_sim no)
-		(in_bom yes)
-		(on_board yes)
-		(dnp no)
-		(fields_autoplaced yes)
-		(property "Reference" "J3"
-			(at 194.31 65.4049 90)
-			(effects
-				(font
-					(size 1.27 1.27)
-				)
-				(justify left)
-			)
-		)
-		(property "Value" "GND"
-			(at 194.31 67.9449 90)
-			(effects
-				(font
-					(size 1.27 1.27)
-				)
-				(justify left)
-			)
-		)
-		(property "Footprint" ""
-			(at 193.04 66.04 0)
-			(effects
-				(font
-					(size 1.27 1.27)
-				)
-				(hide yes)
-			)
-		)
-		(property "Datasheet" "~"
-			(at 193.04 66.04 0)
-			(effects
-				(font
-					(size 1.27 1.27)
-				)
-				(hide yes)
-			)
-		)
-		(property "Description" "Generic connector, single row, 01x01, script generated"
-			(at 193.04 66.04 0)
-			(effects
-				(font
-					(size 1.27 1.27)
-				)
-				(hide yes)
-			)
-		)
-		(pin "1"
-		)
-		(instances
-			(project "VC5_schematic"
-				(path "/236c86f4-0879-4356-88b2-65461f963bd6"
-					(reference "J3")
-					(unit 1)
-				)

Commit message: added missing footprints, changed schematic symbols for the rotaries
Parts:
- J2: footprint (none) -> Connector_PinSocket_2.54mm:PinSocket_1x02_P2.54mm_Vertical
- U1: footprint RPi_Pico:RPi_Pico_SMD_TH -> RPI_Pico_THT:RPi_Pico_SMD_TH
Changed lines of the file:
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@@
 			)
 		)
-		(property "Footprint" ""
+		(property "Footprint" "Connector_PinSocket_2.54mm:PinSocket_1x02_P2.54mm_Vertical"
 			(at 138.43 53.34 0)
 			(effects
@@
 			)
 		)
-		(property "Footprint" "RPi_Pico:RPi_Pico_SMD_TH"
+		(property "Footprint" "RPI_Pico_THT:RPi_Pico_SMD_TH"
 			(at 156.21 95.25 90)
 			(effects
@@
 			)
 		)
-		(property "Datasheet" ""
+		(property "Datasheet" "https://datasheets.raspberrypi.com/pico/pico-datasheet.pdf"
 			(at 156.21 95.25 0)
 			(effects

Commit message: first layout
Parts:
- removed U1: Pico, RPI_Pico_THT:RPi_Pico_SMD_TH, symbol MCU_RaspberryPi_Pico_and_Boards:Pico
- added U1: Pico, RPI_Pico_THT:RPi_Pico_THT, symbol RPI_Pico:Pico
Connections:
- net +3.3V: now also U1.36 (3V3)
- net +5V: now also U1.39 (VSYS), U1.40 (VBUS)
- net CLK: now also U1.24 (GPIO18)
- net CS0: now also U1.16 (GPIO12)
- net CS1: now also U1.17 (GPIO13)
- net CS2: now also U1.19 (GPIO14)
- net CS3: now also U1.22 (GPIO17)
- net CS4: now also U1.20 (GPIO15)
- net DIN: now also U1.25 (GPIO19)
- net DISP_RESET: now also U1.14 (GPIO10)
- net D/C: now also U1.21 (GPIO16)
- net GND: now also U1.13 (GND), U1.18 (GND), U1.23 (GND), U1.28 (GND), U1.3 (GND), U1.38 (GND), U1.8 (GND)
- net I2C_SCL: now also U1.10 (GPIO7)
- net I2C_SDA: now also U1.9 (GPIO6)
- net LED: now also U1.26 (GPIO20)
- net MCP_RESET: now also U1.4 (GPIO2)
- net at J2.1 (Pin_1): now also U1.1 (GPIO0)
- no-connect marks 19 -> 16

Commit message: added MCP interrupt line
Connections:
- net MCP_INT: now reaches U1.5 (GPIO3)
- no-connect marks 16 -> 15
Changed lines of the file:
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@@
-	)
-	(no_connect
-		(at 138.43 81.28)
 	)
 	(no_connect
@@
 	(wire
 		(pts
-			(xy 180.34 116.84) (xy 180.34 153.67)
-		)
-		(stroke
-			(width 0)
-			(type default)
-		)
-	)
-	(wire
-		(pts
 			(xy 173.99 111.76) (xy 200.66 111.76)
 		)
@@
 	(wire
 		(pts
+			(xy 180.34 116.84) (xy 180.34 148.59)
+		)
+		(stroke
+			(width 0)
+			(type default)
+		)
+	)
+	(wire
+		(pts
 			(xy 111.76 104.14) (xy 111.76 148.59)
+		)
+		(stroke
+			(width 0)
+			(type default)
+		)
+	)
+	(wire
+		(pts
+			(xy 121.92 81.28) (xy 138.43 81.28)
 		)
 		(stroke
@@
 			(effects
 				(font
+					(size 1.27 1.27)
+				)
+				(justify right)
+				(hide yes)
+			)
+		)
+	)
+	(global_label "MCP_INT"
+		(shape output)
+		(at 121.92 81.28 180)
+		(fields_autoplaced yes)
+		(effects
+			(font
+				(size 1.27 1.27)
+			)
+			(justify right)
+		)
+		(property "Intersheetrefs" "${INTERSHEET_REFS}"
+			(at 111.7271 81.28 0)
+			(effects
+				(font
